File: PCB/GalaxyModPCB/GalaxyModPCB.kicad_sch (KiCad schematic)
At the start: 53 parts, among them J1 Power Header, J2 Boot mode, J3 LED RGBW Connector, J4 USB to UART, J5 Motor Connector, J6 Projector Connector, Q1 BCP56, Q2 BCP56, Q3 BCP56, Q4 BCP56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

Commit message: Connected all but islands
Parts:
- added J4: JTAG, Jumper:SolderJumper-3_P1.3mm_Open_Pad1.0x1.5mm_NumberLabels, symbol Connector_Generic:Conn_01x04
- renumbered J4 to J5, J5 to J6, J6 to J7
Connections:
- net at U2.13 (IO14): now also J4.1 (Pin_1)
- net at U2.14 (IO12): now also J4.2 (Pin_2)
- net at U2.16 (IO13): now also J4.3 (Pin_3)
- net at U2.23 (IO15): now also J4.4 (Pin_4)
Changed lines of the file:
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@@
+    (stroke (width 0) (type default) (color 0 0 0 0))
+  )
+  (wire (pts (xy 176.53 81.28) (xy 176.53 73.66))
     (stroke (width 0) (type default) (color 0 0 0 0))
   )
@@
     (stroke (width 0) (type default) (color 0 0 0 0))
   )
+  (wire (pts (xy 147.32 81.28) (xy 176.53 81.28))
+    (stroke (width 0) (type default) (color 0 0 0 0))
+  )
   (wire (pts (xy 153.67 66.04) (xy 153.67 134.62))
     (stroke (width 0) (type default) (color 0 0 0 0))
@@
     (stroke (width 0) (type default) (color 0 0 0 0))
   )
+  (wire (pts (xy 147.32 86.36) (xy 179.07 86.36))
+    (stroke (width 0) (type default) (color 0 0 0 0))
+  )
   (wire (pts (xy 40.64 142.24) (xy 40.64 148.59))
     (stroke (width 0) (type default) (color 0 0 0 0))
@@
     (stroke (width 0) (type default) (color 0 0 0 0))
   )
+  (wire (pts (xy 173.99 71.12) (xy 181.61 71.12))
+    (stroke (width 0) (type default) (color 0 0 0 0))
+  )
   (wire (pts (xy 57.15 132.08) (xy 151.13 132.08))
     (stroke (width 0) (type default) (color 0 0 0 0))
@@
     (stroke (width 0) (type default) (color 0 0 0 0))
   )
+  (wire (pts (xy 176.53 73.66) (xy 181.61 73.66))
+    (stroke (width 0) (type default) (color 0 0 0 0))
+  )
   (wire (pts (xy 139.7 180.34) (xy 147.32 180.34))
     (stroke (width 0) (type default) (color 0 0 0 0))
@@
     (stroke (width 0) (type default) (color 0 0 0 0))
   )
+  (wire (pts (xy 171.45 68.58) (xy 181.61 68.58))
+    (stroke (width 0) (type default) (color 0 0 0 0))
+  )
   (wire (pts (xy 147.32 73.66) (xy 168.91 73.66))
     (stroke (width 0) (type default) (color 0 0 0 0))
@@
     (stroke (width 0) (type default) (color 0 0 0 0))
   )
+  (wire (pts (xy 179.07 86.36) (xy 179.07 76.2))
+    (stroke (width 0) (type default) (color 0 0 0 0))
+  )
   (wire (pts (xy 54.61 100.33) (xy 54.61 134.62))
     (stroke (width 0) (type default) (color 0 0 0 0))
@@
     (stroke (width 0) (type default) (color 0 0 0 0))
   )
+  (wire (pts (xy 147.32 78.74) (xy 173.99 78.74))
+    (stroke (width 0) (type default) (color 0 0 0 0))
+  )
   (wire (pts (xy 99.06 176.53) (xy 99.06 173.99))
     (stroke (width 0) (type default) (color 0 0 0 0))
   )
+  (wire (pts (xy 171.45 83.82) (xy 171.45 68.58))
+    (stroke (width 0) (type default) (color 0 0 0 0))
+  )
   (wire (pts (xy 104.14 190.5) (xy 107.95 190.5))
     (stroke (width 0) (type default) (color 0 0 0 0))
@@
     (stroke (width 0) (type default) (color 0 0 0 0))
   )
+  (wire (pts (xy 173.99 78.74) (xy 173.99 71.12))
+    (stroke (width 0) (type default) (color 0 0 0 0))
+  )
   (wire (pts (xy 25.4 166.37) (xy 25.4 160.02))
     (stroke (width 0) (type default) (color 0 0 0 0))
@@
   )
   (wire (pts (xy 156.21 172.72) (xy 156.21 168.91))
+    (stroke (width 0) (type default) (color 0 0 0 0))
+  )
+  (wire (pts (xy 147.32 83.82) (xy 171.45 83.82))
+    (stroke (width 0) (type default) (color 0 0 0 0))
+  )
+  (wire (pts (xy 179.07 76.2) (xy 181.61 76.2))
     (stroke (width 0) (type default) (color 0 0 0 0))
   )
@@
   (symbol (lib_id "Connector_Generic:Conn_01x03") (at 44.45 102.87 180) (unit 1)
     (in_bom yes) (on_board yes) (fields_autoplaced)
-    (property "Reference" "J4" (id 0) (at 44.45 93.98 0))
+    (property "Reference" "J5" (id 0) (at 44.45 93.98 0))
     (property "Value" "USB to UART" (id 1) (at 44.45 96.52 0))
     (property "Footprint" "Jumper:SolderJumper-3_P1.3mm_Open_Pad1.0x1.5mm" (id 2) (at 44.45 102.87 0)
@@
     (pin "2")
   )
+  (symbol (lib_id "Connector_Generic:Conn_01x04") (at 186.69 71.12 0) (unit 1)
+    (in_bom yes) (on_board yes) (fields_autoplaced)
+    (property "Reference" "J4" (id 0) (at 189.23 71.1199 0)
+      (effects (font (size 1.27 1.27)) (justify left))
+    )
+    (property "Value" "JTAG" (id 1) (at 189.23 73.6599 0)
+      (effects (font (size 1.27 1.27)) (justify left))
+    )
+    (property "Footprint" "Jumper:SolderJumper-3_P1.3mm_Open_Pad1.0x1.5mm_NumberLabels" (id 2) (at 186.69 71.12 0)
+      (effects (font (size 1.27 1.27)) hide)
+    )
+    (property "Datasheet" "~" (id 3) (at 186.69 71.12 0)
+      (effects (font (size 1.27 1.27)) hide)
+    )
+    (pin "1")
+    (pin "2")
+    (pin "3")
+    (pin "4")
+  )
   (symbol (lib_id "power:GNDREF") (at 207.01 160.02 0) (unit 1)
     (in_bom yes) (on_board yes)
@@
   (symbol (lib_id "Connector_Generic:Conn_01x02") (at 137.16 175.26 90) (unit 1)
     (in_bom yes) (on_board yes)
-    (property "Reference" "J5" (id 0) (at 135.89 170.18 90)
+    (property "Reference" "J6" (id 0) (at 135.89 170.18 90)
       (effects (font (size 1.27 1.27)) (justify right))
     )
@@
   (symbol (lib_id "Connector_Generic:Conn_01x02") (at 73.66 177.8 90) (unit 1)
     (in_bom yes) (on_board yes)
-    (property "Reference" "J6" (id 0) (at 72.39 172.72 90)
+    (property "Reference" "J7" (id 0) (at 72.39 172.72 90)
       (effects (font (size 1.27 1.27)) (justify right))
     )
@@
       (reference "J3") (unit 1) (value "LED RGBW Connector") (footprint "Connector_PinHeader_2.54mm:PinHeader_1x05_P2.54mm_Vertical")
     )
+    (path "/a9b7e881-7700-43f2-aa69-227b0b4ae11f"
+      (reference "J4") (unit 1) (value "JTAG") (footprint "Jumper:SolderJumper-3_P1.3mm_Open_Pad1.0x1.5mm_NumberLabels")
+    )
     (path "/8053d7a9-b591-4fcc-92bc-dac28827855b"
-      (reference "J4") (unit 1) (value "USB to UART") (footprint "Jumper:SolderJumper-3_P1.3mm_Open_Pad1.0x1.5mm")
+      (reference "J5") (unit 1) (value "USB to UART") (footprint "Jumper:SolderJumper-3_P1.3mm_Open_Pad1.0x1.5mm")
     )
     (path "/b966e064-33c4-411a-9b47-10b81f480fe0"
-      (reference "J5") (unit 1) (value "Motor Connector") (footprint "Connector_PinHeader_2.54mm:PinHeader_1x02_P2.54mm_Vertical")
+      (reference "J6") (unit 1) (value "Motor Connector") (footprint "Connector_PinHeader_2.54mm:PinHeader_1x02_P2.54mm_Vertical")
     )
     (path "/d0bd552a-bfa0-4f1f-b5c2-ee2ac8ffb873"
-      (reference "J6") (unit 1) (value "Projector Connector") (footprint "Connector_PinHeader_2.54mm:PinHeader_1x02_P2.54mm_Vertical")
+      (reference "J7") (unit 1) (value "Projector Connector") (footprint "Connector_PinHeader_2.54mm:PinHeader_1x02_P2.54mm_Vertical")
     )
     (path "/07c21dd4-4418-486e-86c7-56e99ce42fe6"

Commit message: Updated schematic with BJTs
Parts:
- removed Q2, Q3, Q4, Q5, Q6: BCP56, Package_TO_SOT_SMD:SOT-223-3_TabPin2, symbol Transistor_BJT:BCP56
- added Q? (x5): BC817-40-7-F, Package_TO_SOT_SMD:SOT-23, symbol Transistor_BJT:BCP56
- Q1: value BCP56 -> BC817-40-7-F; footprint Package_TO_SOT_SMD:SOT-223-3_TabPin2 -> Package_TO_SOT_SMD:SOT-23
- R10, R12, R14, R17, R19, R8: value 1K -> 270
Connections:
- net GNDREF: now also Q?.3 (E), Q?.3 (E), Q?.3 (E), Q?.3 (E), Q?.3 (E)
- net at R12.2: now also Q?.1 (B)
- net at R14.2: now also Q?.1 (B)
- net at R7.2: now also Q?.2 (C), Q?.4 (C)
- net at R6.2: now also Q?.2 (C), Q?.4 (C)
- net at R5.2: now also Q?.2 (C), Q?.4 (C)
- net at R17.1: now also Q?.1 (B)
- net at D3.2 (A), J6.2 (Pin_2): now also Q?.2 (C), Q?.4 (C)
- net at R19.1: now also Q?.1 (B)
- net at R20.1: now also Q?.2 (C), Q?.4 (C)
- net at R10.2: now also Q?.1 (B)

Commit message: Added resistor to motor
Parts:
- added R?: 200, Resistor_SMD:R_0805_2012Metric_Pad1.20x1.40mm_HandSolder, symbol Device:R_Small
- gave numbers to parts that had none: 5
Connections:
- net at Q5.2 (C), Q5.4 (C): now also R?.1; no longer D3.2 (A), J6.2 (Pin_2)
- new net: D3.2 (A), J6.2 (Pin_2), R?.2
Other:
- moved on the sheet: D3
Changed lines of the file:
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@@
 (kicad_sch (version 20211123) (generator eeschema)
   (paper "A4")
+  (junction (at 140.97 180.34) (diameter 0) (color 0 0 0 0)
+  )
   (junction (at 156.21 161.29) (diameter 0) (color 0 0 0 0)
   )
@@
   (junction (at 129.54 180.34) (diameter 0) (color 0 0 0 0)
   )
-  (junction (at 147.32 180.34) (diameter 0) (color 0 0 0 0)
-  )
   (junction (at 146.05 45.72) (diameter 0) (color 0 0 0 0)
   )
@@
     (stroke (width 0) (type default) (color 0 0 0 0))
   )
-  (wire (pts (xy 147.32 194.31) (xy 142.24 194.31))
-    (stroke (width 0) (type default) (color 0 0 0 0))
-  )
   (wire (pts (xy 115.57 59.69) (xy 115.57 63.5))
     (stroke (width 0) (type default) (color 0 0 0 0))
@@
     (stroke (width 0) (type default) (color 0 0 0 0))
   )
+  (wire (pts (xy 148.59 180.34) (xy 151.13 180.34))
+    (stroke (width 0) (type default) (color 0 0 0 0))
+  )
   (wire (pts (xy 102.87 63.5) (xy 104.14 63.5))
     (stroke (width 0) (type default) (color 0 0 0 0))
@@
     (stroke (width 0) (type default) (color 0 0 0 0))
   )
-  (wire (pts (xy 139.7 180.34) (xy 147.32 180.34))
+  (wire (pts (xy 139.7 180.34) (xy 140.97 180.34))
     (stroke (width 0) (type default) (color 0 0 0 0))
   )
@@
     (stroke (width 0) (type default) (color 0 0 0 0))
   )
-  (wire (pts (xy 147.32 180.34) (xy 147.32 194.31))
+  (wire (pts (xy 140.97 180.34) (xy 140.97 194.31))
     (stroke (width 0) (type default) (color 0 0 0 0))
   )
@@
     (stroke (width 0) (type default) (color 0 0 0 0))
   )
-  (wire (pts (xy 129.54 194.31) (xy 134.62 194.31))
+  (wire (pts (xy 129.54 194.31) (xy 130.81 194.31))
     (stroke (width 0) (type default) (color 0 0 0 0))
   )
@@
     (stroke (width 0) (type default) (color 0 0 0 0))
   )
+  (wire (pts (xy 138.43 194.31) (xy 140.97 194.31))
+    (stroke (width 0) (type default) (color 0 0 0 0))
+  )
   (wire (pts (xy 49.53 102.87) (xy 57.15 102.87))
     (stroke (width 0) (type default) (color 0 0 0 0))
@@
     (stroke (width 0) (type default) (color 0 0 0 0))
   )
+  (wire (pts (xy 140.97 180.34) (xy 143.51 180.34))
+    (stroke (width 0) (type default) (color 0 0 0 0))
+  )
   (wire (pts (xy 223.52 69.85) (xy 242.57 69.85))
     (stroke (width 0) (type default) (color 0 0 0 0))
@@
   )
   (wire (pts (xy 214.63 137.16) (xy 223.52 137.16))
-    (stroke (width 0) (type default) (color 0 0 0 0))
-  )
-  (wire (pts (xy 151.13 180.34) (xy 147.32 180.34))
     (stroke (width 0) (type default) (color 0 0 0 0))
   )
@@
   (symbol (lib_id "Transistor_BJT:BCP56") (at 156.21 177.8 90) (mirror x) (unit 1)
     (in_bom yes) (on_board yes) (fields_autoplaced)
-    (property "Reference" "Q?" (id 0) (at 156.21 184.15 90))
+    (property "Reference" "Q5" (id 0) (at 156.21 184.15 90))
     (property "Value" "BC817-40-7-F" (id 1) (at 156.21 186.69 90))
     (property "Footprint" "Package_TO_SOT_SMD:SOT-23" (id 2) (at 158.115 182.88 0)
@@
   (symbol (lib_id "Transistor_BJT:BCP56") (at 220.98 121.92 0) (unit 1)
     (in_bom yes) (on_board yes) (fields_autoplaced)
-    (property "Reference" "Q?" (id 0) (at 226.06 120.6499 0)
+    (property "Reference" "Q2" (id 0) (at 226.06 120.6499 0)
       (effects (font (size 1.27 1.27)) (justify left))
     )
@@
   (symbol (lib_id "Transistor_BJT:BCP56") (at 236.22 152.4 0) (unit 1)
     (in_bom yes) (on_board yes) (fields_autoplaced)
-    (property "Reference" "Q?" (id 0) (at 241.3 151.1299 0)
+    (property "Reference" "Q4" (id 0) (at 241.3 151.1299 0)
       (effects (font (size 1.27 1.27)) (justify left))
     )
@@
   (symbol (lib_id "Transistor_BJT:BCP56") (at 99.06 187.96 90) (mirror x) (unit 1)
     (in_bom yes) (on_board yes) (fields_autoplaced)
-    (property "Reference" "Q?" (id 0) (at 99.06 194.31 90))
+    (property "Reference" "Q6" (id 0) (at 99.06 194.31 90))
     (property "Value" "BC817-40-7-F" (id 1) (at 99.06 196.85 90))
     (property "Footprint" "Package_TO_SOT_SMD:SOT-23" (id 2) (at 100.965 193.04 0)
@@
     (pin "2")
   )
+  (symbol (lib_id "Device:R_Small") (at 146.05 180.34 270) (unit 1)
+    (in_bom yes) (on_board yes)
+    (property "Reference" "R?" (id 0) (at 146.05 177.8 90))
+    (property "Value" "200" (id 1) (at 146.05 182.88 90))
+    (property "Footprint" "Resistor_SMD:R_0805_2012Metric_Pad1.20x1.40mm_HandSolder" (id 2) (at 146.05 180.34 0)
+      (effects (font (size 1.27 1.27)) hide)
+    )
+    (property "Datasheet" "~" (id 3) (at 146.05 180.34 0)
+      (effects (font (size 1.27 1.27)) hide)
+    )
+    (pin "1")
+    (pin "2")
+  )
   (symbol (lib_id "Switch:SW_Push") (at 33.02 142.24 180) (unit 1)
     (in_bom yes) (on_board yes)
@@
   (symbol (lib_id "Transistor_BJT:BCP56") (at 228.6 137.16 0) (unit 1)
     (in_bom yes) (on_board yes) (fields_autoplaced)
-    (property "Reference" "Q?" (id 0) (at 233.68 135.8899 0)
+    (property "Reference" "Q3" (id 0) (at 233.68 135.8899 0)
       (effects (font (size 1.27 1.27)) (justify left))
     )
@@
     (pin "1")
   )
-  (symbol (lib_id "Device:D_Schottky") (at 138.43 194.31 0) (unit 1)
-    (in_bom yes) (on_board yes)
-    (property "Reference" "D3" (id 0) (at 142.24 191.77 0)
-      (effects (font (size 1.27 1.27)) (justify right))
-    )
-    (property "Value" "Motor" (id 1) (at 140.97 189.23 0)
-      (effects (font (size 1.27 1.27)) (justify right))
-    )
-    (property "Footprint" "Diode_SMD:D_SMA_Handsoldering" (id 2) (at 138.43 194.31 0)
-      (effects (font (size 1.27 1.27)) hide)
-    )
-    (property "Datasheet" "~" (id 3) (at 138.43 194.31 0)
+  (symbol (lib_id "Device:D_Schottky") (at 134.62 194.31 0) (unit 1)
+    (in_bom yes) (on_board yes)
+    (property "Reference" "D3" (id 0) (at 138.43 191.77 0)
+      (effects (font (size 1.27 1.27)) (justify right))
+    )
+    (property "Value" "Motor" (id 1) (at 137.16 189.23 0)
+      (effects (font (size 1.27 1.27)) (justify right))
+    )
+    (property "Footprint" "Diode_SMD:D_SMA_Handsoldering" (id 2) (at 134.62 194.31 0)
+      (effects (font (size 1.27 1.27)) hide)
+    )
+    (property "Datasheet" "~" (id 3) (at 134.62 194.31 0)
       (effects (font (size 1.27 1.27)) hide)
     )
@@
       (reference "Q1") (unit 1) (value "BC817-40-7-F") (footprint "Package_TO_SOT_SMD:SOT-23")
     )
+    (path "/23a89ff5-66a4-4fb3-8361-6570fa9b906b"
+      (reference "Q2") (unit 1) (value "BC817-40-7-F") (footprint "Package_TO_SOT_SMD:SOT-23")
+    )
+    (path "/aeef4a9a-29f5-42ec-84c8-a1cd2e9f35bf"
+      (reference "Q3") (unit 1) (value "BC817-40-7-F") (footprint "Package_TO_SOT_SMD:SOT-23")
+    )
+    (path "/3a5c0131-d5ac-432a-ba39-0c0a8fc351bb"
+      (reference "Q4") (unit 1) (value "BC817-40-7-F") (footprint "Package_TO_SOT_SMD:SOT-23")
+    )
     (path "/1f2fbb51-c6f1-4be2-90d7-da05d7e7bccb"
-      (reference "Q?") (unit 1) (value "BC817-40-7-F") (footprint "Package_TO_SOT_SMD:SOT-23")
-    )
-    (path "/23a89ff5-66a4-4fb3-8361-6570fa9b906b"
-      (reference "Q?") (unit 1) (value "BC817-40-7-F") (footprint "Package_TO_SOT_SMD:SOT-23")
-    )
-    (path "/3a5c0131-d5ac-432a-ba39-0c0a8fc351bb"
-      (reference "Q?") (unit 1) (value "BC817-40-7-F") (footprint "Package_TO_SOT_SMD:SOT-23")
+      (reference "Q5") (unit 1) (value "BC817-40-7-F") (footprint "Package_TO_SOT_SMD:SOT-23")
     )
     (path "/4ed361fe-72fd-4ec5-a53d-925f42f44c7f"
-      (reference "Q?") (unit 1) (value "BC817-40-7-F") (footprint "Package_TO_SOT_SMD:SOT-23")
-    )
-    (path "/aeef4a9a-29f5-42ec-84c8-a1cd2e9f35bf"
-      (reference "Q?") (unit 1) (value "BC817-40-7-F") (footprint "Package_TO_SOT_SMD:SOT-23")
+      (reference "Q6") (unit 1) (value "BC817-40-7-F") (footprint "Package_TO_SOT_SMD:SOT-23")
     )
     (path "/50389375-5435-4213-9da6-292fdec189bf"
@@
       (reference "R20") (unit 1) (value "100") (footprint "Resistor_SMD:R_0805_2012Metric_Pad1.20x1.40mm_HandSolder")
     )
+    (path "/a8bc941f-a6f3-4aa4-83a3-3df84a67ed4c"
+      (reference "R?") (unit 1) (value "200") (footprint "Resistor_SMD:R_0805_2012Metric_Pad1.20x1.40mm_HandSolder")
+    )
     (path "/bd16ea3d-7700-4729-93ff-63f7d5806951"

Commit message: Close data
Parts:
- gave numbers to parts that had none: 1
- renumbered R20 to R21
Changed lines of the file:
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@@
   (symbol (lib_id "Device:R_Small") (at 146.05 180.34 270) (unit 1)
     (in_bom yes) (on_board yes)
-    (property "Reference" "R?" (id 0) (at 146.05 177.8 90))
+    (property "Reference" "R20" (id 0) (at 146.05 177.8 90))
     (property "Value" "200" (id 1) (at 146.05 182.88 90))
     (property "Footprint" "Resistor_SMD:R_0805_2012Metric_Pad1.20x1.40mm_HandSolder" (id 2) (at 146.05 180.34 0)
@@
   (symbol (lib_id "Device:R_Small") (at 81.28 190.5 270) (unit 1)
     (in_bom yes) (on_board yes)
-    (property "Reference" "R20" (id 0) (at 81.28 187.96 90))
+    (property "Reference" "R21" (id 0) (at 81.28 187.96 90))
     (property "Value" "100" (id 1) (at 81.28 193.04 90))
     (property "Footprint" "Resistor_SMD:R_0805_2012Metric_Pad1.20x1.40mm_HandSolder" (id 2) (at 81.28 190.5 0)
@@
       (reference "R19") (unit 1) (value "270") (footprint "Resistor_SMD:R_0805_2012Metric_Pad1.20x1.40mm_HandSolder")
     )
+    (path "/a8bc941f-a6f3-4aa4-83a3-3df84a67ed4c"
+      (reference "R20") (unit 1) (value "200") (footprint "Resistor_SMD:R_0805_2012Metric_Pad1.20x1.40mm_HandSolder")
+    )
     (path "/bb4f8379-181f-4f50-8058-4e4e1b274751"
-      (reference "R20") (unit 1) (value "100") (footprint "Resistor_SMD:R_0805_2012Metric_Pad1.20x1.40mm_HandSolder")
-    )
-    (path "/a8bc941f-a6f3-4aa4-83a3-3df84a67ed4c"
-      (reference "R?") (unit 1) (value "200") (footprint "Resistor_SMD:R_0805_2012Metric_Pad1.20x1.40mm_HandSolder")
+      (reference "R21") (unit 1) (value "100") (footprint "Resistor_SMD:R_0805_2012Metric_Pad1.20x1.40mm_HandSolder")
     )
     (path "/bd16ea3d-7700-4729-93ff-63f7d5806951"

Commit message: Updated resistors for motor control
Parts:
- R17: value 270 -> 4.8K
- R20: value 200 -> 100
Changed lines of the file:
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@@
     (in_bom yes) (on_board yes)
     (property "Reference" "R20" (id 0) (at 146.05 177.8 90))
-    (property "Value" "200" (id 1) (at 146.05 182.88 90))
+    (property "Value" "100" (id 1) (at 146.05 182.88 90))
     (property "Footprint" "Resistor_SMD:R_0805_2012Metric_Pad1.20x1.40mm_HandSolder" (id 2) (at 146.05 180.34 0)
       (effects (font (size 1.27 1.27)) hide)
@@
     (in_bom yes) (on_board yes)
     (property "Reference" "R17" (id 0) (at 151.13 166.37 90))
-    (property "Value" "270" (id 1) (at 153.67 166.37 90))
+    (property "Value" "4.8K" (id 1) (at 153.67 166.37 90))
     (property "Footprint" "Resistor_SMD:R_0805_2012Metric_Pad1.20x1.40mm_HandSolder" (id 2) (at 156.21 166.37 0)
       (effects (font (size 1.27 1.27)) hide)
@@
     )
     (path "/b356be86-93d4-4174-8b16-7626a0f8c2ea"
-      (reference "R17") (unit 1) (value "270") (footprint "Resistor_SMD:R_0805_2012Metric_Pad1.20x1.40mm_HandSolder")
+      (reference "R17") (unit 1) (value "4.8K") (footprint "Resistor_SMD:R_0805_2012Metric_Pad1.20x1.40mm_HandSolder")
     )
     (path "/4acacc10-5bf1-4299-9017-e1f9fedc6f74"
@@
     )
     (path "/a8bc941f-a6f3-4aa4-83a3-3df84a67ed4c"
-      (reference "R20") (unit 1) (value "200") (footprint "Resistor_SMD:R_0805_2012Metric_Pad1.20x1.40mm_HandSolder")
+      (reference "R20") (unit 1) (value "100") (footprint "Resistor_SMD:R_0805_2012Metric_Pad1.20x1.40mm_HandSolder")
     )
     (path "/bb4f8379-181f-4f50-8058-4e4e1b274751"

Commit message: icy layout suggestions
Parts:
- J2: footprint Jumper:SolderJumper-2_P1.3mm_Open_TrianglePad1.0x1.5mm -> Resistor_SMD:R_0805_2012Metric_Pad1.20x1.40mm_HandSolder
- R17: value 4.8K -> 270R
